File: kicad_hello_world.kicad_sch (KiCad schematic)
At the start: 3 parts

Commit message: Finish Part 2
Parts:
- BT1: renamed from BT?; value Battery_Cell -> 3V; footprint (none) -> Battery:BatteryHolder_Keystone_1058_1x2032
- D1: renamed from D?; value LED -> red; footprint (none) -> LED_THT:LED_D5.0mm
- R1: renamed from R?; value R_US -> 1k; footprint (none) -> Resistor_THT:R_Axial_DIN0309_L9.0mm_D3.2mm_P12.70mm_Horizontal
Changed lines of the file:
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@@
     (rev "0")
+  )
+  (junction (at 120.65 116.84) (diameter 0) (color 0 0 0 0)
+  )
+  (junction (at 120.65 93.98) (diameter 0) (color 0 0 0 0)
   )
   (junction (at 134.62 88.9) (diameter 0) (color 0 0 0 0)
@@
     (stroke (width 0) (type default) (color 0 0 0 0))
   )
-  (wire (pts (xy 120.65 101.6) (xy 120.65 88.9))
+  (wire (pts (xy 120.65 101.6) (xy 120.65 93.98))
     (stroke (width 0) (type default) (color 0 0 0 0))
   )
@@
     (stroke (width 0) (type default) (color 0 0 0 0))
   )
-  (wire (pts (xy 120.65 109.22) (xy 120.65 125.73))
+  (wire (pts (xy 120.65 93.98) (xy 120.65 88.9))
+    (stroke (width 0) (type default) (color 0 0 0 0))
+  )
+  (wire (pts (xy 120.65 116.84) (xy 120.65 125.73))
+    (stroke (width 0) (type default) (color 0 0 0 0))
+  )
+  (wire (pts (xy 120.65 109.22) (xy 120.65 116.84))
     (stroke (width 0) (type default) (color 0 0 0 0))
   )
@@
     (effects (font (size 1.27 1.27)) (justify left bottom))
   )
+  (symbol (lib_id "power:PWR_FLAG") (at 120.65 116.84 90) (unit 1)
+    (in_bom yes) (on_board yes) (fields_autoplaced)
+    (property "Reference" "#FLG02" (id 0) (at 118.745 116.84 0)
+      (effects (font (size 1.27 1.27)) hide)
+    )
+    (property "Value" "PWR_FLAG" (id 1) (at 116.84 116.8399 90)
+      (effects (font (size 1.27 1.27)) (justify left))
+    )
+    (property "Footprint" "" (id 2) (at 120.65 116.84 0)
+      (effects (font (size 1.27 1.27)) hide)
+    )
+    (property "Datasheet" "~" (id 3) (at 120.65 116.84 0)
+      (effects (font (size 1.27 1.27)) hide)
+    )
+    (pin "1")
+  )
   (symbol (lib_id "power:VCC") (at 134.62 88.9 0) (unit 1)
     (in_bom yes) (on_board yes) (fields_autoplaced)
-    (property "Reference" "#PWR?" (id 0) (at 134.62 92.71 0)
+    (property "Reference" "#PWR01" (id 0) (at 134.62 92.71 0)
       (effects (font (size 1.27 1.27)) hide)
     )
@@
   (symbol (lib_id "Device:Battery_Cell") (at 120.65 106.68 0) (unit 1)
     (in_bom yes) (on_board yes) (fields_autoplaced)
-    (property "Reference" "BT?" (id 0) (at 124.46 103.3779 0)
+    (property "Reference" "BT1" (id 0) (at 124.46 103.3779 0)
       (effects (font (size 1.27 1.27)) (justify left))
     )
-    (property "Value" "Battery_Cell" (id 1) (at 124.46 105.9179 0)
+    (property "Value" "3V" (id 1) (at 124.46 105.9179 0)
       (effects (font (size 1.27 1.27)) (justify left))
     )
-    (property "Footprint" "" (id 2) (at 120.65 105.156 90)
+    (property "Footprint" "Battery:BatteryHolder_Keystone_1058_1x2032" (id 2) (at 120.65 105.156 90)
       (effects (font (size 1.27 1.27)) hide)
     )
@@
   (symbol (lib_id "Device:R_US") (at 149.86 97.79 0) (unit 1)
     (in_bom yes) (on_board yes) (fields_autoplaced)
-    (property "Reference" "R?" (id 0) (at 152.4 96.5199 0)
+    (property "Reference" "R1" (id 0) (at 152.4 96.5199 0)
       (effects (font (size 1.27 1.27)) (justify left))
     )
-    (property "Value" "R_US" (id 1) (at 152.4 99.0599 0)
+    (property "Value" "1k" (id 1) (at 152.4 99.0599 0)
       (effects (font (size 1.27 1.27)) (justify left))
     )
-    (property "Footprint" "" (id 2) (at 150.876 98.044 90)
+    (property "Footprint" "Resistor_THT:R_Axial_DIN0309_L9.0mm_D3.2mm_P12.70mm_Horizontal" (id 2) (at 150.876 98.044 90)
       (effects (font (size 1.27 1.27)) hide)
     )
@@
     (pin "2")
   )
+  (symbol (lib_id "power:PWR_FLAG") (at 120.65 93.98 90) (unit 1)
+    (in_bom yes) (on_board yes) (fields_autoplaced)
+    (property "Reference" "#FLG01" (id 0) (at 118.745 93.98 0)
+      (effects (font (size 1.27 1.27)) hide)
+    )
+    (property "Value" "PWR_FLAG" (id 1) (at 116.84 93.9799 90)
+      (effects (font (size 1.27 1.27)) (justify left))
+    )
+    (property "Footprint" "" (id 2) (at 120.65 93.98 0)
+      (effects (font (size 1.27 1.27)) hide)
+    )
+    (property "Datasheet" "~" (id 3) (at 120.65 93.98 0)
+      (effects (font (size 1.27 1.27)) hide)
+    )
+    (pin "1")
+  )
   (symbol (lib_id "power:GND") (at 134.62 125.73 0) (unit 1)
     (in_bom yes) (on_board yes) (fields_autoplaced)
-    (property "Reference" "#PWR?" (id 0) (at 134.62 132.08 0)
+    (property "Reference" "#PWR02" (id 0) (at 134.62 132.08 0)
       (effects (font (size 1.27 1.27)) hide)
     )
@@
   (symbol (lib_id "Device:LED") (at 149.86 118.11 90) (unit 1)
     (in_bom yes) (on_board yes) (fields_autoplaced)
-    (property "Reference" "D?" (id 0) (at 153.67 118.4274 90)
+    (property "Reference" "D1" (id 0) (at 153.67 118.4274 90)
       (effects (font (size 1.27 1.27)) (justify right))
     )
-    (property "Value" "LED" (id 1) (at 153.67 120.9674 90)
+    (property "Value" "red" (id 1) (at 153.67 120.9674 90)
       (effects (font (size 1.27 1.27)) (justify right))
     )
-    (property "Footprint" "" (id 2) (at 149.86 118.11 0)
+    (property "Footprint" "LED_THT:LED_D5.0mm" (id 2) (at 149.86 118.11 0)
       (effects (font (size 1.27 1.27)) hide)
     )
@@
   )
   (symbol_instances
+    (path "/a844945d-58d8-4e26-a57e-e4bd91e5534f"
+      (reference "#FLG01") (unit 1) (value "PWR_FLAG") (footprint "")
+    )
+    (path "/1388dcac-ed0c-469b-b688-5fb1fdf0d6d0"
+      (reference "#FLG02") (unit 1) (value "PWR_FLAG") (footprint "")
+    )
     (path "/1f43f476-cb60-420d-9a08-3dbc68764604"
-      (reference "#PWR?") (unit 1) (value "VCC") (footprint "")
+      (reference "#PWR01") (unit 1) (value "VCC") (footprint "")
     )
     (path "/caff1926-2c48-4d7b-bc28-88847424c436"
-      (reference "#PWR?") (unit 1) (value "GND") (footprint "")
+      (reference "#PWR02") (unit 1) (value "GND") (footprint "")
     )
     (path "/28c49f01-b0c2-4cde-b1d7-785e9b8c1f72"
-      (reference "BT?") (unit 1) (value "Battery_Cell") (footprint "")
+      (reference "BT1") (unit 1) (value "3V") (footprint "Battery:BatteryHolder_Keystone_1058_1x2032")
     )
     (path "/fb80a86e-1b7c-49c3-bf6d-6f7eb2345a1f"
-      (reference "D?") (unit 1) (value "LED") (footprint "")
+      (reference "D1") (unit 1) (value "red") (footprint "LED_THT:LED_D5.0mm")
     )
     (path "/57c9b780-6cf7-4c25-9fa1-98ec9e41c534"
-      (reference "R?") (unit 1) (value "R_US") (footprint "")
+      (reference "R1") (unit 1) (value "1k") (footprint "Resistor_THT:R_Axial_DIN0309_L9.0mm_D3.2mm_P12.70mm_Horizontal")
     )
   )
